File: SAQ_KiCad_one/SAQ_KiCad_one.kicad_pcb (KiCad board)
At the start: 2 copper layers, 67 x 54 mm, 58 parts, among them J1 Conn_Coaxial, J2 Conn_Coaxial, J3 Power_IN, J4 Conn_Coaxial, Q1 2SC5095, Q2 2SC5095, SW1 SW_SPDT, U1 MC78L15_TO92, U2 LM79L15_TO92, U3 IVC102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

Commit message: finised second version
Parts:
- removed TP10, TP11, TP3, TP7, TP9: TestPoint_Alt, TestPoint:TestPoint_THTPad_2.5x2.5mm_Drill1.2mm
- added R18: DNP, Resistor_SMD:R_0805_2012Metric_Pad1.20x1.40mm_HandSolder, F.Cu at (167.5, 34.9)
- added R19: 450, Resistor_SMD:R_0805_2012Metric_Pad1.20x1.40mm_HandSolder, F.Cu at (128.4, 29.6)
- added R20: 450, Resistor_SMD:R_0805_2012Metric_Pad1.20x1.40mm_HandSolder, F.Cu at (144.2, 40.3)
- added R21: 450, Resistor_SMD:R_0805_2012Metric_Pad1.20x1.40mm_HandSolder, F.Cu at (164.4, 39.0)
- added R22: 450, Resistor_SMD:R_0805_2012Metric_Pad1.20x1.40mm_HandSolder, F.Cu at (151.2, 37.7)
- added R23: 450, Resistor_SMD:R_0805_2012Metric_Pad1.20x1.40mm_HandSolder, F.Cu at (158.2, 27.1)
- added TEST1: Conn_01x02_Female, Connector_PinHeader_1.00mm:PinHeader_1x02_P1.00mm_Vertical, F.Cu at (128.7, 26.9)
- added TEST2: Conn_01x02_Female, Connector_PinHeader_1.00mm:PinHeader_1x02_P1.00mm_Vertical, F.Cu at (147.2, 40.3)
- added TEST3: Conn_01x02_Female, Connector_PinHeader_1.00mm:PinHeader_1x02_P1.00mm_Vertical, F.Cu at (167.3, 39.0)
- added TEST4: Conn_01x02_Female, Connector_PinHeader_1.00mm:PinHeader_1x02_P1.00mm_Vertical, F.Cu at (154.1, 37.7)
- added TEST5: Conn_01x02_Female, Connector_PinHeader_1.00mm:PinHeader_1x02_P1.00mm_Vertical, F.Cu at (161.4, 27.1)
- C10, C11, C9: moved to B.Cu
- moved TP5 112.3 mm to (108.8, 19.5)
- moved C9 110.0 mm to (139.1, 38.9)
- moved C8 108.8 mm to (136.8, 27.8)
- moved C11 86.1 mm to (158.9, 49.8), turned to 0 degrees
- moved C2 61.6 mm to (164.8, 62.9), turned to 90 degrees
- moved C4 59.9 mm to (160.5, 62.4), turned to 90 degrees
- moved C13 59.1 mm to (157.9, 36.3)
- moved RV1 58.9 mm to (126.6, 62.1), turned to 180 degrees
- moved U4 57.6 mm to (117.8, 51.9)
- moved U1 57.5 mm to (117.8, 58.5)
- moved U2 57.4 mm to (117.8, 64.6)
- moved J4 55.4 mm to (165.9, 19.9)
- moved R6 54.9 mm to (155.0, 56.0), turned to 90 degrees
- moved J3 54.7 mm to (108.9, 55.9)
- moved R5 52.9 mm to (152.5, 55.9)
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Connections:
- J4 pad 2: GNDD -> GND
- U3 pad 13: GNDD -> GND
Routing:
- net -15V: track 0.00 -> 107.3 mm, vias 1 -> 2
- net +15V: track 1.84 -> 107.8 mm, vias 1 -> 2
- net GND: track 42.3 -> 135.0 mm, vias 1 -> 16
- net +9V: track 0.00 -> 86.4 mm, vias 0 -> 2
- net VDD: track 0.00 -> 80.7 mm, vias 0 -> 3
- net +5V: track 3.05 -> 36.0 mm
- net Net-(J3-Pad1): track 0.00 -> 20.5 mm
- net Net-(C12-Pad2): track 40.0 -> 24.8 mm, vias 0 -> 2
- net Net-(J2-Pad1): track 0.00 -> 12.2 mm
- net Net-(R20-Pad2): track 3.20 -> 13.9 mm, vias 1 -> 0
- net Net-(J3-Pad3): track 0.00 -> 8.93 mm
- net GNDD: track 8.74 -> 0.00 mm, vias 1 -> 0
- net Net-(J1-Pad1): track 0.00 -> 6.39 mm
- net Net-(R1-Pad1): track 0.00 -> 5.13 mm
- net Net-(Q1-Pad2): track 6.18 -> 10.8 mm
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- added copper zone on B.Cu, net GND

Commit message: added changes to one and made a remote power board
Parts:
- removed C10, C11: 0.1u, Capacitor_SMD:C_1206_3216Metric_Pad1.33x1.80mm_HandSolder
- removed R13, R14, R15: 1k, Resistor_SMD:R_0805_2012Metric_Pad1.20x1.40mm_HandSolder
- removed U5: TL062, Package_SO:SOIC-8_3.9x4.9mm_P1.27mm
- added JP3: Jumper_2_Open, Jumper:SolderJumper-2_P1.3mm_Open_RoundedPad1.0x1.5mm, F.Cu at (146.8, 30.1)
- added TP3: TestPoint_Alt, TestPoint:TestPoint_THTPad_D4.0mm_Drill2.0mm, F.Cu at (143.4, 19.1)
- TEST1, TEST2, TEST3, TEST4, TEST5: footprint Connector_PinHeader_1.00mm:PinHeader_1x02_P1.00mm_Vertical -> Connector_PinSocket_2.54mm:PinSocket_1x02_P2.54mm_Vertical
- moved TEST4 10.2 mm to (160.6, 29.8)
- moved R22 9.45 mm to (156.5, 29.8)
- moved R12 8.97 mm to (148.6, 42.0), turned to 0 degrees
- moved R21 8.50 mm to (156.5, 42.0)
- moved TEST3 7.38 mm to (160.6, 42.0)
- moved R8 6.67 mm to (148.6, 36.9)
- moved TEST2 6.37 mm to (142.7, 44.8)
- moved R11 6.22 mm to (148.6, 39.4), turned to 180 degrees
- moved R18 6.05 mm to (162.1, 37.5), turned to 270 degrees
- moved R10 4.77 mm to (152.8, 43.0), turned to 90 degrees
- moved C13 4.66 mm to (153.6, 38.2), turned to 270 degrees
- moved R7 4.54 mm to (150.8, 30.1)
- moved U6 2.68 mm to (157.4, 35.3), turned to 90 degrees
- moved JP2 2.15 mm to (146.7, 33.8)
- moved R23 1.97 mm to (156.5, 26.2)
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- renumbered JP2 to JP1, JP1 to JP2
Connections:
- R10 pad 1: Net-(R10-Pad1) -> GND
- R11 pad 1: Net-(R10-Pad2) -> Net-(R11-Pad1)
- R12 pad 2: Net-(R12-Pad2) -> Net-(R10-Pad2)
- R18 pad 1: Net-(R15-Pad2) -> Net-(R10-Pad2)
- R21 pad 2: Net-(R14-Pad2) -> Net-(R10-Pad2)
- R7 pad 1: Net-(R7-Pad1) -> Net-(JP3-Pad2)
- R8 pad 2: Net-(R10-Pad1) -> Net-(R11-Pad1)
- U3 pad 12: Net-(R7-Pad1) -> Net-(JP3-Pad1)
- U6 pad 2: Net-(R15-Pad2) -> Net-(R10-Pad2)
Routing:
- net GND: track 135.0 -> 224.2 mm, vias 16 -> 24
- net -15V: track 107.3 -> 148.5 mm, vias 2 -> 1
- net +15V: track 107.8 -> 81.7 mm, vias 2 -> 1
- net Net-(R14-Pad2): track 12.2 -> 0.00 mm
- net Net-(R10-Pad2): track 5.86 -> 17.1 mm
- net Net-(R13-Pad2): track 9.28 -> 0.00 mm
- net Net-(R7-Pad1): track 9.14 -> 0.00 mm, vias 1 -> 0
- net Net-(JP3-Pad1): track 0.00 -> 8.32 mm, vias 0 -> 1
- net Net-(C12-Pad1): track 18.0 -> 24.7 mm, vias 0 -> 2
- net +9V: track 86.4 -> 92.9 mm, vias 2 -> 1
- net Net-(Q1-Pad2): track 10.8 -> 15.3 mm
- net Net-(R11-Pad2): track 6.74 -> 2.58 mm
- net Net-(R15-Pad2): track 3.63 -> 0.00 mm
- net Net-(C12-Pad2): track 24.8 -> 28.2 mm, vias 2 -> 3
- net Net-(R10-Pad1): track 3.21 -> 0.00 mm
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- added copper zone on GND.Cu, net GND
- removed copper zone on B.Cu, net GND
Other:
- outline, holes or cut-outs redrawn
- copper layers 2 -> 4
- board text added: "+V"
- board text added: "-V"
- board text added: "GND"
