File: SAQ_KiCad_one/SAQ_KiCad_one.sch (KiCad schematic (older format))
At the start: 62 parts, among them J1 Conn_Coaxial, J2 Conn_Coaxial, J3 Power_IN, J4 Conn_Coaxial, Q1 2SC5095, Q2 2SC5095, SW1 SW_SPDT, U1 MC78L15_TO92, U2 LM79L15_TO92, U3 IVC102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

Commit message: finised second version
Parts:
- removed TP10, TP11, TP3, TP7, TP9: TestPoint_Alt, TestPoint:TestPoint_THTPad_2.5x2.5mm_Drill1.2mm, symbol Connector:TestPoint_Alt
- added R18: DNP, Resistor_SMD:R_0805_2012Metric_Pad1.20x1.40mm_HandSolder, symbol Device:R_Small_US
- added R19, R20, R21, R22, R23: 450, Resistor_SMD:R_0805_2012Metric_Pad1.20x1.40mm_HandSolder, symbol Device:R_Small_US
- added TEST1, TEST2, TEST3, TEST4, TEST5: Conn_01x02_Female, Connector_PinHeader_1.00mm:PinHeader_1x02_P1.00mm_Vertical, symbol Connector:Conn_01x02_Female
Connections:
- wire segments 180 -> 190

Commit message: added changes to one and made a remote power board
Parts:
- removed C10, C11: 0.1u, Capacitor_SMD:C_1206_3216Metric_Pad1.33x1.80mm_HandSolder, symbol Device:C_Small
- removed R13, R14, R15: 1k, Resistor_SMD:R_0805_2012Metric_Pad1.20x1.40mm_HandSolder, symbol Device:R_Small_US
- removed U5: TL062, Package_SO:SOIC-8_3.9x4.9mm_P1.27mm, symbol Amplifier_Operational:TL062
- added JP3: Jumper_2_Open, Jumper:SolderJumper-2_P1.3mm_Open_RoundedPad1.0x1.5mm, symbol Jumper:Jumper_2_Open
- added TP3: TestPoint_Alt, TestPoint:TestPoint_THTPad_D4.0mm_Drill2.0mm, symbol Connector:TestPoint_Alt
- TEST1, TEST2, TEST3, TEST4, TEST5: footprint Connector_PinHeader_1.00mm:PinHeader_1x02_P1.00mm_Vertical -> Connector_PinSocket_2.54mm:PinSocket_1x02_P2.54mm_Vertical
- renumbered JP2 to JP1, JP1 to JP2
Connections:
- net GND: now also R10.1, TP3.1
- net at R12.2: now also R10.2, R18.1, R21.2, U6.2 (+)
- net at U3.12 (S2): now also JP3.1 (A); no longer R7.1
- net at R11.1: now also R8.2; no longer R10.2
- new net: JP3.2 (B), R7.1
Other:
- moved on the sheet: C12, C13, J4, R10, R16, R17, R18, R19, R20, R21, R22, R23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
